File: Microcontroladores (Tareas)/micro_puerta/MICROCONTRADOR.kicad_sch (KiCad schematic)
At the start: 1 part, among them U1 ESP32-WROOM-32

Commit message: Actualizacion de micro_puerta
Changed lines of the file:
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@@
+		)
+	)
+	(hierarchical_label "BUZZER_micro"
+		(shape output)
+		(at 83.82 130.81 180)
+		(effects
+			(font
+				(size 1.27 1.27)
+			)
+			(justify right)
 		)
 	)
@@
 		(effects
 			(font
+				(size 1.27 1.27)
+			)
+			(justify right)
+		)
+	)
+	(hierarchical_label "LAMP_micro"
+		(shape output)
+		(at 82.55 116.84 180)
+		(effects
+			(font
