File: Microcontroladores (Tareas)/micro_puerta/POWER_SUPPLY.kicad_sch (KiCad schematic)
At the start: 0 parts

Commit message: Actualizacion de micro_puerta
Parts:
- added C10: 22uF, symbol Device:C_Small
- added C8: 10nF, symbol Device:C_Small
- added C9: 100nF, symbol Device:C_Small
- added L1: L_Iron, symbol Device:L_Iron
- added U4: AP63203WU, Package_TO_SOT_SMD:TSOT-23-6, symbol Regulator_Switching:AP63203WU
Connections:
- net +3.3V: now also C10.1, L1.2, U4.1 (FB)
- net GND: now also C10.2, C8.2, U4.4 (GND)
- net VCC: now also C8.1, U4.2 (EN), U4.3 (IN)
- new net: C9.1, U4.5 (SW)
- new net: C9.2, L1.1, U4.6 (BST)
