File: Microcontroladores (Tareas)/micro_puerta/board_principal.kicad_sch (KiCad schematic)
At the start: 0 parts

Commit message: Actualizacion de micro_puerta
Other:
- added sheet BUZZER_driver (untitled.kicad_sch)
- sheet Driver_lamp ports: added LAMP, LAMP +, LAMP -; removed none
- sheet MICROCONTRADOR ports: added BUZZER_micro, LAMP_micro; removed none
Changed lines of the file:
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@@
-	(wire
-		(pts
-			(xy 170.18 41.91) (xy 180.34 41.91)
-		)
-		(stroke
-			(width 0)
-			(type default)
-		)
-	)
 	(wire
 		(pts
@@
 	(wire
 		(pts
+			(xy 147.32 58.42) (xy 157.48 58.42)
+		)
+		(stroke
+			(width 0)
+			(type default)
+		)
+	)
+	(wire
+		(pts
+			(xy 181.61 55.88) (xy 190.5 55.88)
+		)
+		(stroke
+			(width 0)
+			(type default)
+		)
+	)
+	(wire
+		(pts
+			(xy 147.32 78.74) (xy 157.48 78.74)
+		)
+		(stroke
+			(width 0)
+			(type default)
+		)
+	)
+	(wire
+		(pts
 			(xy 106.68 63.5) (xy 111.76 63.5)
 		)
@@
 	(wire
 		(pts
+			(xy 181.61 60.96) (xy 190.5 60.96)
+		)
+		(stroke
+			(width 0)
+			(type default)
+		)
+	)
+	(wire
+		(pts
+			(xy 181.61 41.91) (xy 190.5 41.91)
+		)
+		(stroke
+			(width 0)
+			(type default)
+		)
+	)
+	(wire
+		(pts
+			(xy 181.61 82.55) (xy 189.23 82.55)
+		)
+		(stroke
+			(width 0)
+			(type default)
+		)
+	)
+	(wire
+		(pts
 			(xy 88.9 43.18) (xy 93.98 43.18)
 		)
@@
 	(wire
 		(pts
-			(xy 170.18 34.29) (xy 180.34 34.29)
-		)
-		(stroke
-			(width 0)
-			(type default)
-		)
-	)
-	(wire
-		(pts
 			(xy 90.17 82.55) (xy 93.98 82.55)
 		)
@@
 	(wire
 		(pts
+			(xy 181.61 76.2) (xy 189.23 76.2)
+		)
+		(stroke
+			(width 0)
+			(type default)
+		)
+	)
+	(wire
+		(pts
 			(xy 147.32 41.91) (xy 157.48 41.91)
+		)
+		(stroke
+			(width 0)
+			(type default)
+		)
+	)
+	(wire
+		(pts
+			(xy 181.61 34.29) (xy 190.5 34.29)
 		)
 		(stroke
@@
 	(hierarchical_label "RS-485-"
 		(shape output)
-		(at 190.5 85.09 0)
+		(at 189.23 101.6 0)
 		(effects
 			(font
@@
 	(hierarchical_label "LAMP+"
 		(shape output)
-		(at 190.5 59.69 0)
+		(at 190.5 55.88 0)
 		(effects
 			(font
@@
 	(hierarchical_label "MA"
 		(shape output)
-		(at 180.34 34.29 0)
+		(at 190.5 34.29 0)
 		(effects
 			(font
@@
 	(hierarchical_label "LAMP-"
 		(shape output)
-		(at 190.5 55.88 0)
+		(at 190.5 60.96 0)
+		(effects
+			(font
+				(size 1.27 1.27)
+			)
+			(justify left)
+		)
+	)
+	(hierarchical_label "BUZZER+"
+		(shape output)
+		(at 189.23 76.2 0)
 		(effects
 			(font
@@
 	(hierarchical_label "MC"
 		(shape output)
-		(at 180.34 41.91 0)
+		(at 190.5 41.91 0)
 		(effects
 			(font
@@
 	(hierarchical_label "RS-485+"
 		(shape output)
-		(at 190.5 82.55 0)
+		(at 189.23 99.06 0)
 		(effects
 			(font
@@
 			)
 			(justify right)
+		)
+	)
+	(hierarchical_label "BUZZER-"
+		(shape output)
+		(at 189.23 82.55 0)
+		(effects
+			(font
+				(size 1.27 1.27)
+			)
+			(justify left)
 		)
 	)
@@
 			)
 		)
+		(pin "LAMP_micro" output
+			(at 147.32 58.42 0)
+			(effects
+				(font
+					(size 1.27 1.27)
+				)
+				(justify right)
+			)
+		)
+		(pin "BUZZER_micro" output
+			(at 147.32 78.74 0)
+			(effects
+				(font
+					(size 1.27 1.27)
+				)
+				(justify right)
+			)
+		)
 		(instances
 			(project "micro_puerta"
 				(path "/dc282be5-e5dc-42c0-bb17-f509e39380eb/6048650d-625a-424f-9cb1-52e32bdac9fd"
 					(page "10")
+				)
+			)
+		)
+	)
+	(sheet
+		(at 157.48 72.39)
+		(size 24.13 12.7)
+		(exclude_from_sim no)
+		(in_bom yes)
+		(on_board yes)
+		(dnp no)
+		(fields_autoplaced yes)
+		(stroke
+			(width 0.1524)
+			(type solid)
+		)
+		(fill
+			(color 0 0 0 0.0000)
+		)
+		(property "Sheetname" "BUZZER_driver"
+			(at 157.48 71.6784 0)
+			(effects
+				(font
+					(size 1.27 1.27)
+				)
+				(justify left bottom)
+			)
+		)
+		(property "Sheetfile" "untitled.kicad_sch"
+			(at 157.48 85.6746 0)
+			(effects
+				(font
+					(size 1.27 1.27)
+				)
+				(justify left top)
+				(hide yes)
+			)
+		)
+		(pin "BUZZER" input
+			(at 157.48 78.74 180)
+			(effects
+				(font
+					(size 1.27 1.27)
+				)
+				(justify left)
+			)
+		)
+		(pin "BUZZER +" output
+			(at 181.61 76.2 0)
+			(effects
+				(font
+					(size 1.27 1.27)
+				)
+				(justify right)
+			)
+		)
+		(pin "BUZZER -" output
+			(at 181.61 82.55 0)
+			(effects
+				(font
+					(size 1.27 1.27)
+				)
+				(justify right)
+			)
+		)
+		(instances
+			(project "micro_puerta"
+				(path "/dc282be5-e5dc-42c0-bb17-f509e39380eb/6048650d-625a-424f-9cb1-52e32bdac9fd"
+					(page "15")
 				)
 			)
@@
 	)
 	(sheet
-		(at 165.1 50.8)
-		(size 12.7 12.7)
+		(at 157.48 52.07)
+		(size 24.13 12.7)
 		(exclude_from_sim no)
 		(in_bom yes)
@@
 		)
 		(property "Sheetname" "Driver_lamp"
-			(at 165.1 50.0884 0)
+			(at 157.48 51.3584 0)
 			(effects
 				(font
@@
 		)
 		(property "Sheetfile" "Driver_lamp.kicad_sch"
-			(at 165.1 64.0846 0)
+			(at 157.48 65.3546 0)
 			(effects
 				(font
@@
 				(justify left top)
 				(hide yes)
+			)
+		)
+		(pin "LAMP +" output
+			(at 181.61 55.88 0)
+			(effects
+				(font
+					(size 1.27 1.27)
+				)
+				(justify right)
+			)
+		)
+		(pin "LAMP -" output
+			(at 181.61 60.96 0)
+			(effects
+				(font
+					(size 1.27 1.27)
+				)
+				(justify right)
+			)
+		)
+		(pin "LAMP" input
+			(at 157.48 58.42 180)
+			(effects
+				(font
+					(size 1.27 1.27)
+				)
+				(justify left)
 			)
 		)
@@
 	)
 	(sheet
-		(at 165.1 76.2)
-		(size 12.7 12.7)
+		(at 157.48 91.44)
+		(size 24.13 12.7)
 		(exclude_from_sim no)
 		(in_bom yes)
@@
 		)
 		(property "Sheetname" "Driver_rs-485"
-			(at 165.1 75.4884 0)
+			(at 157.48 90.7284 0)
 			(effects
 				(font
@@
 		)
 		(property "Sheetfile" "Driver_rs-485.kicad_sch"
-			(at 165.1 89.4846 0)
+			(at 157.48 104.7246 0)
 			(effects
 				(font
@@
 	(sheet
 		(at 157.48 31.75)
-		(size 12.7 12.7)
+		(size 24.13 12.7)
 		(exclude_from_sim no)
 		(in_bom yes)
@@
 		)
 		(pin "MA" output
-			(at 170.18 34.29 0)
+			(at 181.61 34.29 0)
 			(effects
 				(font
@@
 		)
 		(pin "MC" output
-			(at 170.18 41.91 0)
-			(effects
-				(font
+			(at 181.61 41.91 0)
+			(effects
+				(font
