File: Microcontroladores (Tareas)/micro_puerta/untitled.kicad_sch (KiCad schematic)
At the start: 3 parts, among them Q7 NPN, U6 PC817

Commit message: Actualizacion de micro_puerta
Parts:
- removed Q7: NPN, symbol Simulation_SPICE:NPN
- removed R32: 1K, symbol Device:R_US
- removed U6: PC817, Package_DIP:DIP-4_W7.62mm, symbol Isolator:PC817
- added Q8: NPN, symbol Simulation_SPICE:NPN
- added R33: 1K, symbol Device:R_US
- added U5: PC817, Package_DIP:DIP-4_W7.62mm, symbol Isolator:PC817
Connections:
- net GND: now also Q8.3 (E), U5.2
- net VCC: now also U5.4
- new net: R33.1, U5.3
- new net: Q8.2 (B), R33.2
- new net BUZZER: U5.1
- new net BUZZER -: Q8.1 (C)
