File: Microcontroladores (Tareas)/micro_puerta/Driver_lamp.kicad_sch (KiCad schematic)
At the start: 3 parts, among them Q7 NPN, U6 PC817

Commit message: Sexto commit, Actualización de archivos y ADS
Parts:
- renumbered U6 to U?
Changed lines of the file:
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@@
 		(dnp no)
 		(fields_autoplaced yes)
-		(property "Reference" "#PWR053"
+		(property "Reference" "#PWR?"
 			(at 88.9 81.28 0)
 			(effects
@@
 		(pin "1"
 		)
+		(instances
+			(project "micro_puerta"
+				(path "/dc282be5-e5dc-42c0-bb17-f509e39380eb/6048650d-625a-424f-9cb1-52e32bdac9fd/590f8cc4-94e0-49f8-bec8-9ea1f9275301"
+					(reference "#PWR?")
+					(unit 1)
+				)
+			)
+		)
 	)
 	(symbol
@@
 		(dnp no)
 		(fields_autoplaced yes)
-		(property "Reference" "#PWR054"
+		(property "Reference" "#PWR?"
 			(at 114.3 41.91 0)
 			(effects
@@
 		(pin "1"
 		)
+		(instances
+			(project "micro_puerta"
+				(path "/dc282be5-e5dc-42c0-bb17-f509e39380eb/6048650d-625a-424f-9cb1-52e32bdac9fd/590f8cc4-94e0-49f8-bec8-9ea1f9275301"
+					(reference "#PWR?")
+					(unit 1)
+				)
+			)
+		)
 	)
 	(symbol
@@
 		(dnp no)
 		(fields_autoplaced yes)
-		(property "Reference" "U6"
+		(property "Reference" "U?"
 			(at 102.87 45.72 0)
 			(effects
@@
 		(pin "4"
 		)
-	)
+		(instances
+			(project "micro_puerta"
+				(path "/dc282be5-e5dc-42c0-bb17-f509e39380eb/6048650d-625a-424f-9cb1-52e32bdac9fd/590f8cc4-94e0-49f8-bec8-9ea1f9275301"
+					(reference "U?")
+					(unit 1)
+				)
+			)
+		)
+	)
