File: Microcontroladores (Tareas)/micro_puerta/PuenteH.kicad_sch (KiCad schematic)
At the start: 14 parts, among them Q1 NPN, Q2 NPN, Q3 NMOS, Q4 PMOS, Q5 PMOS, Q6 NMOS, U2 SFH617A-1X016, U3 SFH617A-1X016

Commit message: Actualizacion de micro_puerta
Connections:
- net GND: no longer R27.1, R28.2, R29.1, R31.2, U2.3, U3.3
- new net: R27.1, R28.2, U2.3
- new net: R29.1, R31.2, U3.3
Changed lines of the file:
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@@
-	)
-	(junction
-		(at 111.76 96.52)
-		(diameter 0)
-		(color 0 0 0 0)
 	)
 	(junction
@@
 	)
 	(junction
-		(at 152.4 96.52)
-		(diameter 0)
-		(color 0 0 0 0)
-	)
-	(junction
 		(at 110.49 53.34)
 		(diameter 0)
@@
 	)
 	(junction
-		(at 121.92 96.52)
-		(diameter 0)
-		(color 0 0 0 0)
-	)
-	(junction
 		(at 163.83 53.34)
 		(diameter 0)
@@
 		(color 0 0 0 0)
 	)
-	(junction
-		(at 162.56 96.52)
-		(diameter 0)
-		(color 0 0 0 0)
-	)
 	(wire
 		(pts
@@
 	(wire
 		(pts
-			(xy 111.76 107.95) (xy 111.76 96.52)
+			(xy 111.76 93.98) (xy 111.76 107.95)
 		)
 		(stroke
@@
 	(wire
 		(pts
-			(xy 152.4 96.52) (xy 152.4 100.33)
-		)
-		(stroke
-			(width 0)
-			(type default)
-		)
-	)
-	(wire
-		(pts
-			(xy 162.56 96.52) (xy 152.4 96.52)
+			(xy 152.4 87.63) (xy 152.4 100.33)
 		)
 		(stroke
@@
 	(wire
 		(pts
-			(xy 162.56 110.49) (xy 162.56 96.52)
-		)
-		(stroke
-			(width 0)
-			(type default)
-		)
-	)
-	(wire
-		(pts
 			(xy 86.36 57.15) (xy 86.36 66.04)
 		)
@@
 	(wire
 		(pts
-			(xy 121.92 87.63) (xy 121.92 96.52)
+			(xy 121.92 87.63) (xy 121.92 100.33)
 		)
 		(stroke
@@
 	(wire
 		(pts
-			(xy 111.76 96.52) (xy 121.92 96.52)
-		)
-		(stroke
-			(width 0)
-			(type default)
-		)
-	)
-	(wire
-		(pts
 			(xy 110.49 38.1) (xy 110.49 40.64)
 		)
@@
 	(wire
 		(pts
-			(xy 162.56 93.98) (xy 162.56 96.52)
+			(xy 162.56 93.98) (xy 162.56 110.49)
 		)
 		(stroke
@@
 	(wire
 		(pts
-			(xy 111.76 93.98) (xy 111.76 96.52)
-		)
-		(stroke
-			(width 0)
-			(type default)
-		)
-	)
-	(wire
-		(pts
 			(xy 163.83 38.1) (xy 181.61 38.1)
 		)
@@
 	(wire
 		(pts
-			(xy 121.92 96.52) (xy 121.92 100.33)
-		)
-		(stroke
-			(width 0)
-			(type default)
-		)
-	)
-	(wire
-		(pts
 			(xy 187.96 66.04) (xy 187.96 107.95)
 		)
@@
 		)
 		(stroke
-			(width 0)
-			(type default)
-		)
-	)
-	(wire
-		(pts
-			(xy 152.4 87.63) (xy 152.4 96.52)
-		)
-		(stroke

Commit message: Sexto commit, Actualización de archivos y ADS
Parts:
- added R34, R35: 47, symbol Device:R_US
- added R36, R37: 330, symbol Device:R_US
Connections:
- net GND: now also R28.2, R31.2
- net PHA: now also R37.1; no longer U2.1
- net PHC: now also R36.2; no longer U3.1
- net at Q3.2 (G), R28.1: now also R35.2
- net at Q6.2 (G), R31.1: now also R34.2
- net at R27.1, U2.3: now also R35.1; no longer R28.2
- net at R29.1, U3.3: now also R34.1; no longer R31.2
- new net: R36.1, U3.1
- new net: R37.2, U2.1
